File: Hardware/Qwiic/SparkFun_6DoF_ISM330DHCX.sch (EAGLE design)
At the start: 31 parts, among them J1 QWIIC_RIGHT_ANGLE, J2 QWIIC_RIGHT_ANGLE, U1 ISM330DHCX

Commit message: Updates labels on 1x1 to new SPI nomenclature,
* moves pin1 indicator on IC closer to IC
Connections:
- net SDA renamed SDA/PICO
- net SDI_AUX renamed PICO_AUX
- net SDO/SA0 renamed POCI/SA0
- net SDO_AUX renamed POCI_AUX
Other:
- note added: "ISM330DHCX MODES MODE1: Perhipheral-only mode I2C or SPI MODE2: Sensor Hub mode I2C or SPI with controller I2C port MODE 3 and 4: AUX SPI mode I2C and SPI access (Multi-read)"
- note removed: "ISM339DHCX MODES MODE1: Perhipheral-only mode I2C or SPI MODE2: Sensor Hub mode I2C or SPI with controller I2C port MODE 3 and 4: AUX SPI mode I2C and SPI access (Multi-read)"
Changed lines of the file:
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@@
 <text x="135.636" y="113.792" size="1.778" layer="97" font="vector" align="top-left">Cut trace to remove I2C
 pull-up resistors.</text>
-<text x="20.32" y="109.22" size="1.778" layer="97" font="vector" align="top-left">ISM339DHCX MODES
+<text x="20.32" y="109.22" size="1.778" layer="97" font="vector" align="top-left">ISM330DHCX MODES
 MODE1:  Perhipheral-only mode
    I2C or SPI
@@
 </segment>
 </net>
-<net name="SDA" class="0">
+<net name="SDA/PICO" class="0">
 <segment>
 <wire x1="76.2" y1="144.78" x2="81.28" y2="144.78" width="0.1524" layer="91"/>
@@
 </segment>
 </net>
-<net name="SDO/SA0" class="0">
+<net name="POCI/SA0" class="0">
 <segment>
 <wire x1="76.2" y1="137.16" x2="81.28" y2="137.16" width="0.1524" layer="91"/>
@@
 </segment>
 </net>
-<net name="SDI_AUX" class="0">
+<net name="PICO_AUX" class="0">
 <segment>
 <pinref part="JP3" gate="G$1" pin="5"/>
@@
 </segment>
 </net>
-<net name="SDO_AUX" class="0">
+<net name="POCI_AUX" class="0">
 <segment>
 <wire x1="76.2" y1="129.54" x2="81.28" y2="129.54" width="0.1524" layer="91"/>

Commit message: Moves some vias, fixes "x", "y", and "z" on axes, fixes some schematic typos
Other:
- note added: "Cut traces to remove I2C pull-up resistors."
- note removed: "Cut trace to remove I2C pull-up resistors."
- moved on the sheet: SCX
Changed lines of the file:
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@@
 <text x="243.84" y="88.646" size="1.778" layer="97" font="vector" rot="R180" align="top-left">If using Mode 2 (Sensor Hub Mode),
 cut both traces. </text>
-<text x="135.636" y="113.792" size="1.778" layer="97" font="vector" align="top-left">Cut trace to remove I2C
+<text x="135.636" y="113.792" size="1.778" layer="97" font="vector" align="top-left">Cut traces to remove I2C
 pull-up resistors.</text>
 <text x="20.32" y="109.22" size="1.778" layer="97" font="vector" align="top-left">ISM330DHCX MODES
@@
 <attribute name="VALUE" x="205.74" y="96.52" size="1.778" layer="96" font="vector"/>
 </instance>
-<instance part="GND2" gate="1" x="220.98" y="99.06" smashed="yes">
-<attribute name="VALUE" x="218.44" y="96.52" size="1.778" layer="96" font="vector"/>
+<instance part="GND2" gate="1" x="228.6" y="99.06" smashed="yes">
+<attribute name="VALUE" x="226.06" y="96.52" size="1.778" layer="96" font="vector"/>
 </instance>
 <instance part="SDX" gate="G$1" x="208.28" y="109.22" smashed="yes" rot="R90">
 <attribute name="NAME" x="205.74" y="109.22" size="1.778" layer="95" font="vector" rot="R180"/>
 </instance>
-<instance part="SCX" gate="G$1" x="220.98" y="109.22" smashed="yes" rot="R90">
-<attribute name="NAME" x="218.44" y="109.22" size="1.778" layer="95" font="vector" rot="R180"/>
+<instance part="SCX" gate="G$1" x="228.6" y="109.22" smashed="yes" rot="R90">
+<attribute name="NAME" x="226.06" y="109.22" size="1.778" layer="95" font="vector" rot="R180"/>
 </instance>
 <instance part="LOGO3" gate="G$1" x="190.5" y="33.02" smashed="yes"/>
@@
 <pinref part="GND2" gate="1" pin="GND"/>
 <pinref part="SCX" gate="G$1" pin="1"/>
-<wire x1="220.98" y1="101.6" x2="220.98" y2="104.14" width="0.1524" layer="91"/>
+<wire x1="228.6" y1="101.6" x2="228.6" y2="104.14" width="0.1524" layer="91"/>
 </segment>
 <segment>
@@
 <segment>
 <pinref part="SCX" gate="G$1" pin="2"/>
-<wire x1="220.98" y1="114.3" x2="220.98" y2="116.84" width="0.1524" layer="91"/>
-<wire x1="220.98" y1="116.84" x2="223.52" y2="116.84" width="0.1524" layer="91"/>
-<label x="223.52" y="116.84" size="1.27" layer="95" font="vector" xref="yes"/>
-</segment>
-</net>
+<wire x1="228.6" y1="114.3" x2="228.6" y2="116.84" width="0.1524" layer="91"/>
+<wire x1="228.6" y1="116.84" x2="231.14" y2="116.84" width="0.1524" layer="91"/>
+<label x="231.14" y="116.84" size="1.27" layer="95" font="vector" xref="yes"/>
+</segment>
+</net>
