File: Hardware/Qwiic/SparkFun_6DoF_ISM330DHCX.sch (EAGLE design)
At the start: 31 parts, among them J1 QWIIC_RIGHT_ANGLE, J2 QWIIC_RIGHT_ANGLE, U1 ISM330DHCX

Commit message: Fixes swapped silk on PICO and CS headers, changes to v10, adds "default" text to default address
Other:
- note added: "(Default)"
- note added: "v10"
- note removed: "v01"
Changed lines of the file:
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@@
 <text x="48.006" y="152.654" size="1.27" layer="97" font="vector">VDD Range: 1.71V - 3.6V
 VDDIO Range: 1.62V - 3.6V</text>
-<text x="238.76" y="7.62" size="2.54" layer="94" font="vector">v01</text>
+<text x="238.76" y="7.62" size="2.54" layer="94" font="vector">v10</text>
 <text x="177.8" y="180.34" size="2.54" layer="94" font="vector" align="center">Jumpers</text>
 <text x="152.4" y="129.54" size="1.778" layer="97" font="vector">Cut trace to
@@
 <wire x1="213.36" y1="139.7" x2="213.36" y2="134.62" width="0.2032" layer="97"/>
 <wire x1="213.36" y1="134.62" x2="220.98" y2="134.62" width="0.2032" layer="97"/>
-<wire x1="220.98" y1="134.62" x2="236.22" y2="134.62" width="0.2032" layer="97"/>
-<wire x1="236.22" y1="134.62" x2="236.22" y2="139.7" width="0.2032" layer="97"/>
-<wire x1="236.22" y1="139.7" x2="236.22" y2="144.78" width="0.2032" layer="97"/>
-<wire x1="236.22" y1="144.78" x2="236.22" y2="149.86" width="0.2032" layer="97"/>
-<wire x1="236.22" y1="149.86" x2="236.22" y2="154.94" width="0.2032" layer="97"/>
-<wire x1="236.22" y1="154.94" x2="213.36" y2="154.94" width="0.2032" layer="97"/>
+<wire x1="220.98" y1="134.62" x2="246.38" y2="134.62" width="0.2032" layer="97"/>
+<wire x1="246.38" y1="134.62" x2="246.38" y2="139.7" width="0.2032" layer="97"/>
+<wire x1="246.38" y1="139.7" x2="246.38" y2="144.78" width="0.2032" layer="97"/>
+<wire x1="246.38" y1="144.78" x2="246.38" y2="149.86" width="0.2032" layer="97"/>
+<wire x1="246.38" y1="149.86" x2="246.38" y2="154.94" width="0.2032" layer="97"/>
+<wire x1="246.38" y1="154.94" x2="213.36" y2="154.94" width="0.2032" layer="97"/>
 <wire x1="213.36" y1="149.86" x2="220.98" y2="149.86" width="0.2032" layer="97"/>
-<wire x1="220.98" y1="149.86" x2="236.22" y2="149.86" width="0.2032" layer="97"/>
+<wire x1="220.98" y1="149.86" x2="246.38" y2="149.86" width="0.2032" layer="97"/>
 <wire x1="220.98" y1="149.86" x2="220.98" y2="144.78" width="0.2032" layer="97"/>
 <wire x1="220.98" y1="144.78" x2="220.98" y2="139.7" width="0.2032" layer="97"/>
 <wire x1="220.98" y1="139.7" x2="220.98" y2="134.62" width="0.2032" layer="97"/>
-<wire x1="220.98" y1="144.78" x2="236.22" y2="144.78" width="0.2032" layer="97"/>
-<wire x1="220.98" y1="139.7" x2="236.22" y2="139.7" width="0.2032" layer="97"/>
+<wire x1="220.98" y1="144.78" x2="246.38" y2="144.78" width="0.2032" layer="97"/>
+<wire x1="220.98" y1="139.7" x2="246.38" y2="139.7" width="0.2032" layer="97"/>
 <wire x1="220.98" y1="144.78" x2="213.36" y2="144.78" width="0.2032" layer="97"/>
 <wire x1="213.36" y1="139.7" x2="220.98" y2="139.7" width="0.2032" layer="97"/>
@@
 <wire x1="210.82" y1="152.4" x2="209.804" y2="151.638" width="0.2032" layer="97" style="dashdot"/>
 <text x="167.894" y="11.176" size="2.54" layer="94" font="vector">Elias Santistevan</text>
+<text x="232.41" y="146.558" size="1.778" layer="97" font="vector">(Default)</text>
 </plain>
 <instances>

Commit message: Adds a via, adds some clearer text to the schematic
Other:
- note added: "I2C Address (selectable): 0x6B (Default)"
- moved on the sheet: ADDR, D1, I2C_PU, LED, R1, R2, R4, R5, R6
