File: Hardware/Micro/SparkFun_6DoF_ISM330DHCX_Micro.sch (EAGLE design)
At the start: 25 parts, among them U1 ISM330DHCX

Commit message: Updates labels on Qwiic Micro, Updates IC on Qwiic Micro and Micro
Connections:
- net SDA renamed SDA/PICO
- net SDI_AUX renamed PICO_AUX
- net SDO/SA0 renamed POCI/SA0
- net SDO_AUX renamed POCI_AUX
Changed lines of the file:
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@@
 </segment>
 </net>
-<net name="SDA" class="0">
+<net name="SDA/PICO" class="0">
 <segment>
 <wire x1="76.2" y1="144.78" x2="81.28" y2="144.78" width="0.1524" layer="91"/>
@@
 </segment>
 </net>
-<net name="SDO/SA0" class="0">
+<net name="POCI/SA0" class="0">
 <segment>
 <wire x1="76.2" y1="137.16" x2="81.28" y2="137.16" width="0.1524" layer="91"/>
@@
 </segment>
 </net>
-<net name="SDI_AUX" class="0">
+<net name="PICO_AUX" class="0">
 <segment>
 <pinref part="JP3" gate="G$1" pin="5"/>
@@
 </segment>
 </net>
-<net name="SDO_AUX" class="0">
+<net name="POCI_AUX" class="0">
 <segment>
 <wire x1="76.2" y1="129.54" x2="81.28" y2="129.54" width="0.1524" layer="91"/>
@@
 <pinref part="JP3" gate="G$1" pin="6"/>
 <wire x1="45.72" y1="17.78" x2="50.8" y2="17.78" width="0.1524" layer="91"/>
-<label x="50.8" y="17.78" size="1.27" layer="95" xref="yes"/>
-</segment>
-</net>
+<label x="50.8" y="17.78" size="1.27" layer="95" font="vector" xref="yes"/>
+</segment>
+</net>

Commit message: Fixes labels, realigns the SDX jumper on top
Other:
- note added: "Cut traces to remove I2C pull-up resistors."
- note removed: "Cut trace to remove I2C pull-up resistors."
- moved on the sheet: SCX
Changed lines of the file:
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@@
 <text x="243.84" y="88.646" size="1.778" layer="97" font="vector" rot="R180" align="top-left">If using Mode 2 (Sensor Hub Mode),
 cut both traces. </text>
-<text x="135.636" y="113.792" size="1.778" layer="97" font="vector" align="top-left">Cut trace to remove I2C
+<text x="135.636" y="113.792" size="1.778" layer="97" font="vector" align="top-left">Cut traces to remove I2C
 pull-up resistors.</text>
 <text x="20.32" y="109.22" size="1.778" layer="97" font="vector" align="top-left">ISM330DHCX MODES
@@
 <attribute name="VALUE" x="205.74" y="96.52" size="1.778" layer="96" font="vector"/>
 </instance>
-<instance part="GND2" gate="1" x="220.98" y="99.06" smashed="yes">
-<attribute name="VALUE" x="218.44" y="96.52" size="1.778" layer="96" font="vector"/>
+<instance part="GND2" gate="1" x="226.06" y="99.06" smashed="yes">
+<attribute name="VALUE" x="223.52" y="96.52" size="1.778" layer="96" font="vector"/>
 </instance>
 <instance part="SDX" gate="G$1" x="208.28" y="109.22" smashed="yes" rot="R90">
 <attribute name="NAME" x="205.74" y="109.22" size="1.778" layer="95" font="vector" rot="R180"/>
 </instance>
-<instance part="SCX" gate="G$1" x="220.98" y="109.22" smashed="yes" rot="R90">
-<attribute name="NAME" x="218.44" y="109.22" size="1.778" layer="95" font="vector" rot="R180"/>
+<instance part="SCX" gate="G$1" x="226.06" y="109.22" smashed="yes" rot="R90">
+<attribute name="NAME" x="223.52" y="109.22" size="1.778" layer="95" font="vector" rot="R180"/>
 </instance>
 <instance part="JP3" gate="G$1" x="40.64" y="25.4" smashed="yes" rot="MR180">
@@
 <pinref part="GND2" gate="1" pin="GND"/>
 <pinref part="SCX" gate="G$1" pin="1"/>
-<wire x1="220.98" y1="101.6" x2="220.98" y2="104.14" width="0.1524" layer="91"/>
+<wire x1="226.06" y1="101.6" x2="226.06" y2="104.14" width="0.1524" layer="91"/>
 </segment>
 <segment>
@@
 <segment>
 <pinref part="SCX" gate="G$1" pin="2"/>
-<wire x1="220.98" y1="114.3" x2="220.98" y2="116.84" width="0.1524" layer="91"/>
-<wire x1="220.98" y1="116.84" x2="223.52" y2="116.84" width="0.1524" layer="91"/>
-<label x="223.52" y="116.84" size="1.27" layer="95" font="vector" xref="yes"/>
-</segment>
-</net>
+<wire x1="226.06" y1="114.3" x2="226.06" y2="116.84" width="0.1524" layer="91"/>
+<wire x1="226.06" y1="116.84" x2="228.6" y2="116.84" width="0.1524" layer="91"/>
+<label x="228.6" y="116.84" size="1.27" layer="95" font="vector" xref="yes"/>
+</segment>
+</net>
