File: Hardware/Qwiic Micro Alternate/SparkFun_6DoF_ISM330DHCX_Qwiic_Micro_Alternate.sch (EAGLE design)
At the start: 26 parts, among them J1 Qwiic Right Angle, U1 ISM330DHCX

Commit message: Removes unused size
Parts:
- J2: device SparkFun-Connectors:CONN_021X02_NO_SILK -> SparkFun-Connectors:CONN_02_1.5MM
- TP1, TP2, TP3: value TEST-POINTTP_15TH_THRU -> TEST-POINT3; device SparkFun-Connectors:TEST-POINTTP_15TH_THRU -> SparkFun-Connectors:TEST-POINT3
Changed lines of the file:
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@@
 <part name="LOGO1" library="SparkFun-Aesthetics" deviceset="QWIIC_LOGO" device="_3MM"/>
 <part name="LOGO3" library="SparkFun-Aesthetics" deviceset="SFE_LOGO_NAME_FLAME" device="BLANK"/>
-<part name="J2" library="SparkFun-Connectors" deviceset="CONN_02" device="1X02_NO_SILK"/>
+<part name="J2" library="SparkFun-Connectors" deviceset="CONN_02" device="_1.5MM"/>
 <part name="GND1" library="SparkFun-PowerSymbols" deviceset="GND" device=""/>
-<part name="TP1" library="SparkFun-Connectors" deviceset="TEST-POINT" device="TP_15TH_THRU"/>
-<part name="TP2" library="SparkFun-Connectors" deviceset="TEST-POINT" device="TP_15TH_THRU"/>
-<part name="TP3" library="SparkFun-Connectors" deviceset="TEST-POINT" device="TP_15TH_THRU"/>
+<part name="TP1" library="SparkFun-Connectors" deviceset="TEST-POINT" device="3" value="TEST-POINT3"/>
+<part name="TP2" library="SparkFun-Connectors" deviceset="TEST-POINT" device="3" value="TEST-POINT3"/>
+<part name="TP3" library="SparkFun-Connectors" deviceset="TEST-POINT" device="3" value="TEST-POINT3"/>
 <part name="SUPPLY6" library="SparkFun-PowerSymbols" deviceset="3.3V" device=""/>
 </parts>
