File: Hardware/Qwiic Micro/SparkFun_6DoF_ISM330DHCX_Qwiic_Micro.brd (EAGLE design)
At the start: 19.1 x 7.6 mm, 42 parts, among them J1 Qwiic Right Angle, U1 ISM330DHCX

Commit message: Updates INT2 to rounded, and changes INT text on Micro to INT1
Parts:
- U$11: device top:#INT#21 -> top:#INT1#2
- U$5: device top:#INT#20 -> top:#INT1#0
- moved U$11 0.25 mm to (2.67, 1.27)
- moved U$5 0.25 mm to (2.67, 1.27)
Changed lines of the file:
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@@
 <wire x1="0" y1="0" x2="19.05" y2="0" width="0.2032" layer="20"/>
 <wire x1="19.05" y1="0" x2="19.05" y2="7.62" width="0.2032" layer="20"/>
-<text x="0.263525" y="0.371475" size="0.8128" layer="16" font="vector" ratio="22" rot="SMR90">v10</text>
+<text x="0.263525" y="3.546475" size="0.8128" layer="16" font="vector" ratio="22" rot="SMR90">v10</text>
 <rectangle x1="9.1948" y1="4.953" x2="9.2456" y2="5.1816" layer="41"/>
 <dimension x1="2.54" y1="3.81" x2="0" y2="3.81" x3="1.27" y3="12.7" textsize="1.778" layer="47" dtype="horizontal" unit="inch"/>
@@
 <attribute name="VALUE" x="8.255" y="2.594" size="0.6096" layer="27" font="vector" ratio="20" rot="R180" align="top-center"/>
 </element>
-<element name="U$5" library="top" package="#INT#20" value="" x="2.921" y="1.27" smashed="yes"/>
-<element name="U$11" library="top" package="#INT#21" value="" x="2.921" y="1.27" smashed="yes" rot="MR0"/>
 <element name="U$4" library="top" package="#GND#4" value="" x="2.667" y="6.35" smashed="yes"/>
 <element name="U$10" library="top" package="#GND#4" value="" x="2.667" y="6.35" smashed="yes" rot="MR0"/>
+<element name="U$5" library="top" package="#INT1#0" value="" x="2.667" y="1.27" smashed="yes"/>
+<element name="U$11" library="top" package="#INT1#2" value="" x="2.667" y="1.27" smashed="yes" rot="MR0"/>
 </elements>
 <signals>

Commit message: Renames production files to include version number, updates 0402 RED LED with one that has PROD_ID
Parts:
- D1: device ISM330DHCX:0402-TIGHT -> SparkFun-LED:LED-0402
Changed lines of the file:
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@@
 <element name="FD1" library="SparkFun-Aesthetics" package="FIDUCIAL-MICRO" value="FIDUCIALUFIDUCIAL" x="15.9766" y="6.985" smashed="yes" rot="MR0"/>
 <element name="FD2" library="SparkFun-Aesthetics" package="FIDUCIAL-MICRO" value="FIDUCIALUFIDUCIAL" x="0.6604" y="3.0734" smashed="yes" rot="MR0"/>
-<element name="D1" library="ISM330DHCX" package="0402-TIGHT" value="RED" x="10.0076" y="6.9088" smashed="yes">
+<element name="D1" library="SparkFun-LED" package="LED-0402" value="RED" x="10.0076" y="6.9088" smashed="yes">
 <attribute name="NAME" x="10.0076" y="7.5438" size="0.6096" layer="25" font="vector" ratio="20" align="bottom-center"/>
+<attribute name="PROD_ID" value="DIO-16757" x="10.0076" y="6.9088" size="1.778" layer="27" display="off"/>
 <attribute name="VALUE" value="RED" x="10.0076" y="6.9088" size="1.778" layer="27" display="off"/>
 </element>
